File: nRF24/PCBs/ProgrammingAdapter/ProgrammingAdapter.kicad_sch (KiCad schematic)
At the start: 16 parts, among them J2 5V Out, J3 IIC 3V3, J4 WS2812, J6 SPI Prog, SW1 PA3, SW2 RESET, U1 NRF24L01, U2 ATtiny84, U3 MCP1700x-330

Commit message: LED Strip Controller and Programming Adapter WIP
Parts:
- added C3: 100uF, Capacitor_THT:CP_Radial_D7.5mm_P2.50mm, symbol Device:C_Polarized
- J2: renamed from J6; footprint (none) -> hagego:JST_XH_1x04_P2.54
- J3: footprint (none) -> hagego:JST_XH_1x04_P2.54
- J4: footprint (none) -> hagego:JST_XH_1x03_P2.54
- SW1: footprint Button_Switch_THT:Push_E-Switch_KS01Q01 -> hagego:Micro_Push_Button_6x6
- SW2: footprint Button_Switch_THT:SW_Push_2P1T_Toggle_CK_PVA1xxH1xxxxxxV2 -> hagego:Micro_Push_Button_6x6
- U2: footprint Package_DIP:DIP-14_W7.62mm_Socket -> hagego:Engineering_DIP14_Socket
- renumbered J2 to J1
Connections:
- net GND: now also A1.4 (GND), SW2.2, C3.2
- net MISO: now also A1.15 (D12)
- net MOSI: now also A1.14 (D11)
- net SCK: now also A1.16 (D13)
- net SCL: now also J3.3 (Pin_3), U2.12 (PA1)
- net SDA: now also J3.4 (Pin_4), U2.11 (PA2)
- net at A1.13 (D10): now also J2.1 (Pin_1), SW2.3 (K), SW2.4 (A), U2.4 (~{RESET}/PB3)
- net at A1.3 (~{RESET}): now also C3.1
- net +5V: now reaches A1.30 (VIN)
- net at SW1.3 (K): now also SW1.4 (A), U2.10 (PA3)
- no-connect marks 1 -> 23

Commit message: Programming Adapter production version 1.0
Parts:
- added J5: AM312, hagego:JST_XH_1x03_P2.54, symbol Connector:Conn_01x03_Pin
Connections:
- net GND: now also J5.2 (Pin_2)
- net Vbat: now also J5.1 (Pin_1)
- net at U2.2 (XTAL1/PB0): now also J5.3 (Pin_3)
Changed lines of the file:
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@@
+	)
+	(junction
+		(at 123.19 161.29)
+		(diameter 0)
+		(color 0 0 0 0)
 	)
 	(junction
@@
 		(color 0 0 0 0)
 	)
+	(junction
+		(at 130.81 163.83)
+		(diameter 0)
+		(color 0 0 0 0)
+	)
 	(no_connect
 		(at 76.2 72.39)
@@
 	(wire
 		(pts
+			(xy 109.22 175.26) (xy 130.81 175.26)
+		)
+		(stroke
+			(width 0)
+			(type default)
+		)
+	)
+	(wire
+		(pts
 			(xy 165.1 69.85) (xy 146.05 69.85)
 		)
@@
 	(wire
 		(pts
+			(xy 130.81 163.83) (xy 130.81 175.26)
+		)
+		(stroke
+			(width 0)
+			(type default)
+		)
+	)
+	(wire
+		(pts
 			(xy 146.05 63.5) (xy 146.05 69.85)
 		)
@@
 	(wire
 		(pts
+			(xy 60.96 34.29) (xy 60.96 36.83)
+		)
+		(stroke
+			(width 0)
+			(type default)
+		)
+	)
+	(wire
+		(pts
 			(xy 196.85 44.45) (xy 198.12 44.45)
 		)
@@
 	(wire
 		(pts
+			(xy 123.19 161.29) (xy 123.19 172.72)
+		)
+		(stroke
+			(width 0)
+			(type default)
+		)
+	)
+	(wire
+		(pts
 			(xy 142.24 53.34) (xy 157.48 53.34)
 		)
@@
 	(wire
 		(pts
+			(xy 149.86 71.12) (xy 142.24 71.12)
+		)
+		(stroke
+			(width 0)
+			(type default)
+		)
+	)
+	(wire
+		(pts
 			(xy 109.22 161.29) (xy 123.19 161.29)
 		)
@@
 	(wire
 		(pts
+			(xy 123.19 172.72) (xy 109.22 172.72)
+		)
+		(stroke
+			(width 0)
+			(type default)
+		)
+	)
+	(wire
+		(pts
 			(xy 165.1 105.41) (xy 165.1 69.85)
 		)
@@
 	(wire
 		(pts
+			(xy 109.22 177.8) (xy 149.86 177.8)
+		)
+		(stroke
+			(width 0)
+			(type default)
+		)
+	)
+	(wire
+		(pts
 			(xy 27.94 59.69) (xy 27.94 35.56)
 		)
@@
 		(pts
 			(xy 66.04 114.3) (xy 76.2 114.3)
+		)
+		(stroke
+			(width 0)
+			(type default)
+		)
+	)
+	(wire
+		(pts
+			(xy 149.86 71.12) (xy 149.86 177.8)
 		)
 		(stroke
@@
 	)
 	(symbol
-		(lib_id "power:+5V")
-		(at 60.96 36.83 0)
-		(unit 1)
-		(exclude_from_sim no)
-		(in_bom yes)
-		(on_board yes)
-		(dnp no)
-		(fields_autoplaced yes)
-		(property "Reference" "#PWR02"
-			(at 60.96 40.64 0)
-			(effects
-				(font
-					(size 1.27 1.27)
-				)
-				(hide yes)
-			)
-		)
-		(property "Value" "+5V"
-			(at 60.96 31.75 0)
-			(effects
-				(font
-					(size 1.27 1.27)
-				)
-			)
-		)
-		(property "Footprint" ""
-			(at 60.96 36.83 0)
-			(effects
-				(font
-					(size 1.27 1.27)
-				)
-				(hide yes)
-			)
-		)
-		(property "Datasheet" ""
-			(at 60.96 36.83 0)
-			(effects
-				(font
-					(size 1.27 1.27)
-				)
-				(hide yes)
-			)
-		)
-		(property "Description" "Power symbol creates a global label with name \"+5V\""
-			(at 60.96 36.83 0)
-			(effects
-				(font
-					(size 1.27 1.27)
-				)
-				(hide yes)
-			)
-		)
-		(pin "1"
-		)
-		(instances
-			(project ""
-				(path "/c0b25fac-ce5c-4c3e-a3ea-c1cb16b4e65b"
-					(reference "#PWR02")
-					(unit 1)
-				)
-			)
-		)
-	)
-	(symbol
 		(lib_id "Device:C_Small")
 		(at 179.07 38.1 0)
@@
 					(unit 1)
 				)
+			)
+		)
+	)
+	(symbol
+		(lib_id "power:+5V")
+		(at 60.96 34.29 0)
+		(unit 1)
+		(exclude_from_sim no)
+		(in_bom yes)
+		(on_board yes)
+		(dnp no)
+		(property "Reference" "#PWR02"
+			(at 60.96 38.1 0)
+			(effects
+				(font
+					(size 1.27 1.27)
+				)
+				(hide yes)
+			)
+		)
+		(property "Value" "+5V"
+			(at 60.96 30.226 0)
+			(effects
+				(font
+					(size 1.27 1.27)
+				)
+			)
+		)
+		(property "Footprint" ""
+			(at 60.96 34.29 0)
+			(effects
+				(font
+					(size 1.27 1.27)
+				)
+				(hide yes)
+			)
+		)
+		(property "Datasheet" ""
+			(at 60.96 34.29 0)
+			(effects
+				(font
+					(size 1.27 1.27)
+				)
+				(hide yes)
+			)
+		)
+		(property "Description" "Power symbol creates a global label with name \"+5V\""
+			(at 60.96 34.29 0)
+			(effects
+				(font
+					(size 1.27 1.27)
+				)
+				(hide yes)
+			)
+		)
+		(pin "1"
+		)
+		(instances
+			(project ""
+				(path "/c0b25fac-ce5c-4c3e-a3ea-c1cb16b4e65b"
+					(reference "#PWR02")
+					(unit 1)
+				)
+			)
+		)
+	)
+	(symbol
+		(lib_id "Connector:Conn_01x03_Pin")
+		(at 104.14 175.26 0)
+		(unit 1)
+		(exclude_from_sim no)
+		(in_bom yes)
+		(on_board yes)
+		(dnp no)
+		(property "Reference" "J5"
+			(at 98.806 172.72 0)
+			(effects
+				(font
+					(size 1.27 1.27)
+				)
+			)
+		)
+		(property "Value" "AM312"
+			(at 98.806 175.514 0)
+			(effects
+				(font
+					(size 1.27 1.27)
+				)
+			)
+		)
+		(property "Footprint" "hagego:JST_XH_1x03_P2.54"
+			(at 104.14 175.26 0)
+			(effects
+				(font
+					(size 1.27 1.27)
+				)
+				(hide yes)
+			)
+		)
+		(property "Datasheet" "~"
+			(at 104.14 175.26 0)
+			(effects
+				(font
+					(size 1.27 1.27)
+				)
+				(hide yes)
+			)
+		)
+		(property "Description" "Generic connector, single row, 01x03, script generated"
+			(at 104.14 175.26 0)
+			(effects
+				(font
+					(size 1.27 1.27)
+				)
+				(hide yes)
+			)
+		)
+		(pin "1"
+		)
+		(pin "3"
+		)
+		(pin "2"
+		)
+		(instances
+			(project "ProgrammingAdapter"
+				(path "/c0b25fac-ce5c-4c3e-a3ea-c1cb16b4e65b"
+					(reference "J5")
+					(unit 1)
+				)
