File: nRF24/PCBs/MultiClientSmall/MultiClientSmall.kicad_pcb (KiCad board)
At the start: 2 copper layers, 38 x 38 mm, 21 parts, among them J1 Prog, M1 TP4056, SW1 Button, U1 NRF24L01, U2 ATtiny84, U3 MCP1700x-330, U4 BH1750, U5 AM312, U6 BME280

Commit message: Fixed AM312 motion sensor orientation
Parts:
- renumbered R2 to 100k, R3 to 1M, R1 to 470k
Routing:
- net GND: track 191.6 -> 186.0 mm
- net /VCC: track 114.2 -> 109.4 mm
Changed lines of the file:
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@@
 		)
 	)
-	(property "Version" "1.1")
+	(property "Version" "1.2")
 	(net 0 "")
 	(net 1 "unconnected-(SW1-Pad2)")
@@
 		)
 		(pad "1" thru_hole circle
-			(at -2.54 -1.872 270)
+			(at 2.54 -1.872 270)
 			(size 2 2)
 			(drill 0.8)
@@
 		)
 		(pad "3" thru_hole circle
-			(at 2.54 -1.872 270)
+			(at -2.54 -1.872 270)
 			(size 2 2)
 			(drill 0.8)
@@
 		(descr "Resistor, Axial_DIN0207 series, Axial, Horizontal, pin pitch=10.16mm, 0.25W = 1/4W, length*diameter=6.3*2.5mm^2, http://cdn-reichelt.de/documents/datenblatt/B400/1_4W%23YAG.pdf")
 		(tags "Resistor Axial_DIN0207 series Axial Horizontal pin pitch 10.16mm 0.25W = 1/4W length 6.3mm diameter 2.5mm")
-		(property "Reference" "R3"
+		(property "Reference" "1M"
 			(at 5.08 0 0)
 			(layer "F.SilkS")
@@
 		(descr "Resistor, Axial_DIN0207 series, Axial, Horizontal, pin pitch=10.16mm, 0.25W = 1/4W, length*diameter=6.3*2.5mm^2, http://cdn-reichelt.de/documents/datenblatt/B400/1_4W%23YAG.pdf")
 		(tags "Resistor Axial_DIN0207 series Axial Horizontal pin pitch 10.16mm 0.25W = 1/4W length 6.3mm diameter 2.5mm")
-		(property "Reference" "R2"
+		(property "Reference" "100k"
 			(at 3.81 0 90)
 			(layer "B.SilkS")
@@
 		(descr "Resistor, Axial_DIN0207 series, Axial, Horizontal, pin pitch=10.16mm, 0.25W = 1/4W, length*diameter=6.3*2.5mm^2, http://cdn-reichelt.de/documents/datenblatt/B400/1_4W%23YAG.pdf")
 		(tags "Resistor Axial_DIN0207 series Axial Horizontal pin pitch 10.16mm 0.25W = 1/4W length 6.3mm diameter 2.5mm")
-		(property "Reference" "R1"
+		(property "Reference" "470k"
 			(at 5.08 0 0)
 			(layer "B.SilkS")
@@
 	)
 	(segment
+		(start 150.97 117.348)
+		(end 150.97 117.602)
+		(width 0.5)
+		(layer "F.Cu")
+		(net 5)
+	)
+	(segment
 		(start 137.314 114.084)
 		(end 144 107.398)
@@
 	)
 	(segment
+		(start 150.872 117.348)
+		(end 150.872 109.224)
+		(width 0.3)
+		(layer "F.Cu")
+		(net 5)
+	)
+	(segment
 		(start 121.158 113.284)
 		(end 122.682 113.284)
@@
 	)
 	(segment
+		(start 150.872 109.224)
+		(end 152.146 107.95)
+		(width 0.3)
+		(layer "F.Cu")
+		(net 5)
+	)
+	(segment
 		(start 132.175646 112.262)
 		(end 133.914 114.000354)
@@
 	)
 	(segment
-		(start 150.97 122.428)
-		(end 150.97 122.174)
-		(width 0.5)
-		(layer "B.Cu")
-		(net 5)
-	)
-	(segment
 		(start 153.029694 133.82)
 		(end 149.29528 133.82)
@@
 	)
 	(segment
-		(start 153.497 108.476)
-		(end 152.971 107.95)
-		(width 0.5)
-		(layer "B.Cu")
-		(net 5)
-	)
-	(segment
-		(start 150.97 122.174)
-		(end 153.497 119.647)
-		(width 0.5)
-		(layer "B.Cu")
-		(net 5)
-	)
-	(segment
 		(start 145.03943 128.318)
 		(end 135.37657 128.318)
@@
 	)
 	(segment
-		(start 153.497 119.647)
-		(end 153.497 108.476)
-		(width 0.5)
-		(layer "B.Cu")
-		(net 5)
-	)
-	(segment
 		(start 138.938 129.794)
 		(end 137.462 128.318)
@@
 	)
 	(segment
-		(start 120.142 110.236)
-		(end 121.119 111.213)
-		(width 0.5)
-		(layer "F.Cu")
-		(net 7)
-	)
-	(segment
-		(start 145.542 134.112)
-		(end 145.542 133.858)
+		(start 150.872 122.428)
+		(end 153.162 124.718)
 		(width 0.5)
 		(layer "F.Cu")
@@
 	)
 	(segment
-		(start 153.162 119.794)
-		(end 153.162 131.318)
+		(start 120.142 110.236)
+		(end 121.119 111.213)
 		(width 0.5)
 		(layer "F.Cu")
@@
 	)
 	(segment
-		(start 150.97 117.348)
-		(end 150.97 117.602)
+		(start 145.542 134.112)
+		(end 145.542 133.858)
 		(width 0.5)
 		(layer "F.Cu")
@@
 	)
 	(segment
-		(start 150.97 117.602)
-		(end 153.162 119.794)
-		(width 0.5)
-		(layer "F.Cu")
-		(net 7)
-	)
-	(segment
 		(start 119.634 109.3)
 		(end 120.142 109.808)
@@
 	)
 	(segment
+		(start 153.162 124.718)
+		(end 153.162 131.318)
+		(width 0.5)
+		(layer "F.Cu")
+		(net 7)
+	)
+	(segment
 		(start 129.071 111.213)
 		(end 130.556 109.728)
@@
 	)
 	(segment
+		(start 150.97 122.428)
+		(end 150.97 122.174)
+		(width 0.5)
+		(layer "B.Cu")
+		(net 7)
+	)
+	(segment
 		(start 134.176 127.14672)
 		(end 134.076 127.04672)
@@
 		(polygon
 			(pts
-				(xy 116.84 100.838) (xy 116.84 139.192) (xy 155.194 139.192) (xy 155.194 100.838)
+				(xy 116.84 100.838) (xy 116.84 139.192) (xy 155.194 139.192) (xy 154.94 100.584)
 			)
 		)

Commit message: nRF24 Multi-Client PCB V1.3
Parts:
- removed JP1: CSN, Connector_PinHeader_2.54mm:PinHeader_1x02_P2.54mm_Vertical
- 1M1: renamed from 470k; value 470k -> 1M
- 220k1: renamed from 100k; value 100k -> 220k
- M1: footprint hagego:TP4056-18650 -> KiCad Library:TP4056-18650
- SW1: value Button -> SW_Push_Dual
Connections:
- 1M pad 2: Net-(JP1-B) -> Net-(U1-~{CSN})
- U1 pad 4: Net-(JP1-B) -> Net-(U1-~{CSN})
- U2 pad 5: Net-(JP1-A) -> Net-(U1-~{CSN})
Routing:
- net Net-(U1-~{CSN}): track 0.00 -> 37.0 mm, vias 0 -> 1
- net Net-(JP1-A): track 32.1 -> 0.00 mm, vias 1 -> 0
- net Net-(JP1-B): track 17.0 -> 0.00 mm
- added copper zone on B.Cu, net GND
- added copper zone on F.Cu, net GND
- removed copper zone on B.Cu, net (none)
- removed copper zone on F.Cu, net (none)
