File: nRF24/PCBs/MultiClientSmall/MultiClientSmall.kicad_sch (KiCad schematic)
At the start: 11 parts, among them M1 TP4056, SW1 SW_Push_Dual, U1 NRF24L01, U2 ATtiny84, U3 MCP1700x-330, U4 BH1750

Commit message: Created MultiClientSmall KiCAD Project
Parts:
- added U5: AM312, hagego:AM312, symbol hagego:AM312
Connections:
- net GND: now also U5.3 (GND)
- net VCC: now also U5.1 (VCC)
- net at U2.2 (XTAL1/PB0): now also U5.2 (VOUT)
Changed lines of the file:
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@@
 		(color 0 0 0 0)
 	)
+	(junction
+		(at 175.26 133.35)
+		(diameter 0)
+		(color 0 0 0 0)
+	)
+	(junction
+		(at 185.42 123.19)
+		(diameter 0)
+		(color 0 0 0 0)
+	)
 	(wire
 		(pts
@@
 	(wire
 		(pts
+			(xy 152.4 104.14) (xy 157.48 104.14)
+		)
+		(stroke
+			(width 0)
+			(type default)
+		)
+	)
+	(wire
+		(pts
 			(xy 162.56 60.96) (xy 162.56 66.04)
 		)
@@
 	(wire
 		(pts
+			(xy 157.48 144.78) (xy 193.04 144.78)
+		)
+		(stroke
+			(width 0)
+			(type default)
+		)
+	)
+	(wire
+		(pts
 			(xy 204.47 77.47) (xy 205.74 77.47)
 		)
@@
 	(wire
 		(pts
+			(xy 175.26 133.35) (xy 175.26 147.32)
+		)
+		(stroke
+			(width 0)
+			(type default)
+		)
+	)
+	(wire
+		(pts
+			(xy 185.42 142.24) (xy 193.04 142.24)
+		)
+		(stroke
+			(width 0)
+			(type default)
+		)
+	)
+	(wire
+		(pts
 			(xy 95.25 93.98) (xy 93.98 93.98)
 		)
@@
 	(wire
 		(pts
+			(xy 175.26 147.32) (xy 193.04 147.32)
+		)
+		(stroke
+			(width 0)
+			(type default)
+		)
+	)
+	(wire
+		(pts
 			(xy 175.26 133.35) (xy 193.04 133.35)
 		)
@@
 	(wire
 		(pts
+			(xy 157.48 104.14) (xy 157.48 144.78)
+		)
+		(stroke
+			(width 0)
+			(type default)
+		)
+	)
+	(wire
+		(pts
 			(xy 83.82 99.06) (xy 95.25 99.06)
 		)
@@
 		(pts
 			(xy 93.98 125.73) (xy 113.03 125.73)
+		)
+		(stroke
+			(width 0)
+			(type default)
+		)
+	)
+	(wire
+		(pts
+			(xy 185.42 123.19) (xy 185.42 142.24)
 		)
 		(stroke
@@
 					(unit 1)
 				)
+			)
+		)
+	)
+	(symbol
+		(lib_id "hagego:AM312")
+		(at 196.85 144.78 0)
+		(unit 1)
+		(exclude_from_sim no)
+		(in_bom yes)
+		(on_board yes)
+		(dnp no)
+		(fields_autoplaced yes)
+		(property "Reference" "U5"
+			(at 203.2 143.5099 0)
+			(effects
+				(font
+					(size 1.27 1.27)
+				)
+				(justify left)
+			)
+		)
+		(property "Value" "AM312"
+			(at 203.2 146.0499 0)
+			(effects
+				(font
+					(size 1.27 1.27)
+				)
+				(justify left)
+			)
+		)
+		(property "Footprint" "hagego:AM312"
+			(at 196.85 144.78 0)
+			(effects
+				(font
+					(size 1.27 1.27)
+				)
+				(hide yes)
+			)
+		)
+		(property "Datasheet" ""
+			(at 196.85 144.78 0)
+			(effects
+				(font
+					(size 1.27 1.27)
+				)
+				(hide yes)
+			)
+		)
+		(property "Description" ""
+			(at 196.85 144.78 0)
+			(effects
+				(font
+					(size 1.27 1.27)
+				)
+				(hide yes)
+			)
+		)
+		(pin "1"
+		)
+		(pin "2"
+		)
+		(pin "3"
+		)
+		(instances
+			(project ""
+				(path "/c0b25fac-ce5c-4c3e-a3ea-c1cb16b4e65b"
+					(reference "U5")
+					(unit 1)
+				)

Commit message: Production Version of nRF24 Multi Client Small
Parts:
- added J1: Prog, Connector_PinHeader_2.54mm:PinHeader_1x04_P2.54mm_Vertical, symbol Connector_Generic:Conn_01x04
- added JP1: CSN, Connector_PinHeader_2.54mm:PinHeader_1x02_P2.54mm_Vertical, symbol Jumper:Jumper_2_Bridged
- added PV1: 6V, hagego:JST_PH_1x02_P2.00, symbol Device:Battery_Cell
- added R3: 1M, Resistor_THT:R_Axial_DIN0207_L6.3mm_D2.5mm_P10.16mm_Horizontal, symbol Device:R
- added U6: BME280, hagego:BME280, symbol hagego:BME280_Module
- Bat1: renamed from BT1; footprint Connector_JST:JST_PH_B2B-PH-K_1x02_P2.00mm_Vertical -> hagego:JST_PH_1x02_P2.00
Connections:
- net GND: now also M1.2 (In-), PV1.2 (-), U6.2 (GND)
- net VCC: now also R3.1, U6.1 (VCC)
- net at U1.4 (~{CSN}): now also JP1.2 (B), R3.2; no longer U2.5 (PB2)
- net SCK: now reaches U1.5 (SCK), U2.9 (PA4)
- net SCK: now also J1.4 (Pin_4)
- net MISO: now reaches U1.6 (MOSI), U2.8 (PA5)
- net MISO: now also J1.3 (Pin_3)
- net MOSI: now reaches U1.7 (MISO), U2.7 (PA6)
- net MOSI: now also J1.2 (Pin_2)
- net SDA: now reaches U2.11 (PA2), U4.4 (SDA)
- net SDA: now also U6.4 (SDA)
- net SCL: now reaches U2.12 (PA1), U4.3 (SCL)
- net SCL: now also U6.3 (SCL)
- net at U2.4 (~{RESET}/PB3): now also J1.1 (Pin_1)
- net +3V7: now reaches Bat1.1 (+), M1.5 (B+)
- net +6V: now reaches M1.1 (In+)
- net +6V: now also PV1.1 (+)
- new net: JP1.1 (A), U2.5 (PB2)
- no-connect marks 0 -> 4
Other:
- title: nRF24 Button -> nRF24 Multi Client
- moved on the sheet: Bat1, C1, C2, M1, R1, R2, SW1, U1, U2, U3, U4, U5

Commit message: Fixed AM312 motion sensor orientation
Parts:
- renumbered R2 to 100k, R1 to 470k
Changed lines of the file:
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@@
 		(dnp no)
 		(fields_autoplaced yes)
-		(property "Reference" "R1"
+		(property "Reference" "470k"
 			(at 154.94 53.3399 0)
 			(effects
@@
 			(project ""
 				(path "/c0b25fac-ce5c-4c3e-a3ea-c1cb16b4e65b"
-					(reference "R1")
+					(reference "470k")
 					(unit 1)
 				)
@@
 		(dnp no)
 		(fields_autoplaced yes)
-		(property "Reference" "R2"
+		(property "Reference" "100k"
 			(at 154.94 63.4999 0)
 			(effects
@@
 			(project ""
 				(path "/c0b25fac-ce5c-4c3e-a3ea-c1cb16b4e65b"
-					(reference "R2")
-					(unit 1)
-				)
+					(reference "100k")
+					(unit 1)
+				)

Commit message: nRF24 Multi-Client PCB V1.3
Parts:
- removed JP1: CSN, Connector_PinHeader_2.54mm:PinHeader_1x02_P2.54mm_Vertical, symbol Jumper:Jumper_2_Bridged
- 1M1: renamed from 470k; value 470k -> 1M
- 220k1: renamed from 100k; value 100k -> 220k
Connections:
- net at R3.2, U1.4 (~{CSN}): now also U2.5 (PB2)
