File: nRF24/PCBs/ESP2nRF24/ESP2nRF24/ESP2nRF24.kicad_pcb (KiCad board)
At the start: 2 copper layers, 68 x 42 mm, 8 parts, among them U1 WEMOS_D1_mini, U2 NRF24L01_Breakout, U3 AM312, U4 BE680, U5 BH1750

Commit message: Changed nRF242ESp local sensor pin to D0
Parts:
- moved C1 6.02 mm to (163.5, 67.6)
Connections:
- U1 pad 11: Net-(U1-D4) -> unconnected-(U1-D4-Pad11)
- U1 pad 3: unconnected-(U1-D0-Pad3) -> Net-(U1-D0)
- U3 pad 2: Net-(U1-D4) -> Net-(U1-D0)
Routing:
- net Net-(U1-D0): track 0.00 -> 71.5 mm, vias 0 -> 2
- net Net-(U1-D4): track 31.5 -> 0.00 mm, vias 1 -> 0
- net Net-(U1-3V3): track 116.1 -> 119.3 mm
- net GND: track 121.9 -> 120.1 mm
- added copper zone on B.Cu, net GND
- added copper zone on F.Cu, net GND
- removed copper zone on B.Cu, net (none)
- removed copper zone on F.Cu, net (none)
