File: nRF24/PCBs/ESP2nRF24/ESP2nRF24/ESP2nRF24.kicad_sch (KiCad schematic)
At the start: 6 parts, among them U1 WEMOS_D1_mini, U2 NRF24L01_Breakout, U3 AM312, U4 BE680, U5 BH1750

Commit message: Changed nRF242ESp local sensor pin to D0
Connections:
- net at U3.2 (VOUT): now also U1.3 (D0); no longer U1.11 (D4)
